File: I2C_Expander/i2c_exapnder/i2c_exapnder.kicad_sch (KiCad schematic)
At the start: 8 parts, among them J1 Conn_01x10, J2 Conn_01x05, J4 Conn_01x05, J5 Conn_01x05

Commit message: Add logo and text to I2C Expander
Other:
- title: (none) -> Kevinbot v3 I2C Expander w/ MPU
Changed lines of the file:
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@@
 (kicad_sch (version 20230121) (generator eeschema)
   (paper "A4")
+  (title_block
+    (title "Kevinbot v3 I2C Expander w/ MPU")
+    (rev "A")
+  )
   (wire (pts (xy 76.2 64.77) (xy 76.2 62.23))
     (stroke (width 0) (type default))
