File: P2 Kevinbot Board.kicad_pcb (KiCad board)
At the start: 2 copper layers, 196.5 x 95.4 mm, 56 parts, among them J11 Screw_Terminal_01x02, J13 Screw_Terminal_01x02, J14 Screw_Terminal_01x02, J17 Conn_01x02, J2 Conn_02x06_Odd_Even, J20 Conn_02x06_Odd_Even, J23 Conn_02x06_Odd_Even, J24 Conn_01x04, J25 Conn_01x04, J26 Conn_01x04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

Commit message: Silkscreen updates
Parts:
- U4: value PCA9685PW -> PCA9685
Other:
- board text added: "A0"
- board text added: "A1"
- board text added: "A2"
- board text added: "A3"
- board text added: "A4"
- board text added: "A5"
- board text added: "E.RST"
- board text added: "PropPlug Programming Header (#32201)"
- board text added: "RESET"
- board text added: "S0"
- board text added: "S1"
- board text added: "S10"
- board text added: "S11"
- board text added: "S12"
- board text added: "S13"
- board text added: "S14"
- board text added: "S15"
- board text added: "S2"
- board text added: "S3"
- board text added: "S4"
- board text added: "S5"
- board text added: "S6"
- board text added: "S7"
- board text added: "S8"
- board text added: "S9"
- board text removed: "RST"
Changed lines of the file:
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@@
     (property "ki_keywords" "PWM LED driver I2C TSSOP")
     (attr smd)
-    (fp_text reference "U4" (at 0 -3.485) (layer "F.SilkS")
-        (effects (font (size 1 1) (thickness 0.15)))
-    )
-    (fp_text value "PCA9685PW" (at 0 5.8) (layer "F.Fab") hide
+    (fp_text reference "U4" (at 0 -3.485) (layer "F.SilkS") hide
+        (effects (font (size 1 1) (thickness 0.15)))
+    )
+    (fp_text value "PCA9685" (at 0 0.325 90) (layer "F.SilkS")
         (effects (font (size 1 1) (thickness 0.15)))
     )
@@
       (net 22 "-BATT") (pinfunction "1") (pintype "input"))
   )
+  (gr_rect (start 66.179 71.125) (end 88.404 81.285)
+    (stroke (width 0.15) (type default)) (fill none) (layer "F.SilkS"))
   (gr_rect (start 65.9445 55.17) (end 262.4535 150.58)
     (stroke (width 0.15) (type solid)) (fill none) (layer "Edge.Cuts"))
@@
     (effects (font (size 1.5 1.5) (thickness 0.3)) (justify bottom))
   )
+  (gr_text "A1" (at 225.183 99.192 90) (layer "F.SilkS")
+    (effects (font (size 1.5 1.5) (thickness 0.3)))
+  )
+  (gr_text "S8" (at 249.059 114.432) (layer "F.SilkS")
+    (effects (font (size 1.5 1.5) (thickness 0.15)) (justify left bottom))
+  )
   (gr_text "LED POWER" (at 106.184 74.935) (layer "F.SilkS")
     (effects (font (size 2 2) (thickness 0.3) bold) (justify bottom))
@@
     (effects (font (size 2 2) (thickness 0.3)) (justify left bottom))
   )
+  (gr_text "S3" (at 249.059 98.176) (layer "F.SilkS")
+    (effects (font (size 1.5 1.5) (thickness 0.15)) (justify left bottom))
+  )
+  (gr_text "S11" (at 247.535 122.052) (layer "F.SilkS")
+    (effects (font (size 1.5 1.5) (thickness 0.15)) (justify left bottom))
+  )
   (gr_text "G" (at 184.289 67.315) (layer "F.SilkS")
     (effects (font (size 1.5 1.5) (thickness 0.3)) (justify bottom))
@@
     (effects (font (size 2.2 2.2) (thickness 0.4) bold) (justify right bottom))
   )
+  (gr_text "A3" (at 225.183 111.384 90) (layer "F.SilkS")
+    (effects (font (size 1.5 1.5) (thickness 0.3)))
+  )
   (gr_text "+" (at 80.149 109.225) (layer "F.SilkS")
     (effects (font (size 2 2) (thickness 0.3)) (justify left bottom))
   )
+  (gr_text "S12" (at 247.535 126.624) (layer "F.SilkS")
+    (effects (font (size 1.5 1.5) (thickness 0.15)) (justify left bottom))
+  )
   (gr_text "BATT 1" (at 85.864 104.78 90) (layer "F.SilkS")
     (effects (font (size 2 2) (thickness 0.3)) (justify bottom))
@@
     (effects (font (size 2 2) (thickness 0.3)) (justify bottom))
   )
+  (gr_text "S0" (at 249.059 90.556) (layer "F.SilkS")
+    (effects (font (size 1.5 1.5) (thickness 0.15)) (justify left bottom))
+  )
+  (gr_text "S14" (at 247.535 131.704) (layer "F.SilkS")
+    (effects (font (size 1.5 1.5) (thickness 0.15)) (justify left bottom))
+  )
+  (gr_text "S6" (at 249.059 107.828) (layer "F.SilkS")
+    (effects (font (size 1.5 1.5) (thickness 0.15)) (justify left bottom))
+  )
   (gr_text "T" (at 176.669 67.315) (layer "F.SilkS")
     (effects (font (size 1.5 1.5) (thickness 0.3)) (justify bottom))
   )
+  (gr_text "S1" (at 249.059 93.096) (layer "F.SilkS")
+    (effects (font (size 1.5 1.5) (thickness 0.15)) (justify left bottom))
+  )
+  (gr_text "+" (at 255.409 88.016) (layer "F.SilkS")
+    (effects (font (size 1.2 1.2) (thickness 0.15)) (justify left bottom))
+  )
+  (gr_text "S10" (at 247.535 119.512) (layer "F.SilkS")
+    (effects (font (size 1.5 1.5) (thickness 0.15)) (justify left bottom))
+  )
+  (gr_text "RESET" (at 124.889 111.13) (layer "F.SilkS")
+    (effects (font (size 2 2) (thickness 0.3)) (justify bottom))
+  )
   (gr_text "BATT 2" (at 85.864 120.655 90) (layer "F.SilkS")
     (effects (font (size 2 2) (thickness 0.3)) (justify bottom))
   )
+  (gr_text "S4" (at 249.059 102.748) (layer "F.SilkS")
+    (effects (font (size 1.5 1.5) (thickness 0.15)) (justify left bottom))
+  )
+  (gr_text "S2" (at 249.059 95.636) (layer "F.SilkS")
+    (effects (font (size 1.5 1.5) (thickness 0.15)) (justify left bottom))
+  )
   (gr_text "-" (at 80.149 87.635) (layer "F.SilkS")
     (effects (font (size 2 2) (thickness 0.3)) (justify left bottom))
   )
-  (gr_text "RST" (at 185.559 71.76) (layer "F.SilkS")
+  (gr_text "A2" (at 225.183 105.288 90) (layer "F.SilkS")
+    (effects (font (size 1.5 1.5) (thickness 0.3)))
+  )
+  (gr_text "E.RST" (at 185.559 71.76) (layer "F.SilkS")
     (effects (font (size 2 2) (thickness 0.3)) (justify bottom))
+  )
+  (gr_text "-" (at 257.949 88.016) (layer "F.SilkS")
+    (effects (font (size 1.2 1.2) (thickness 0.15)) (justify left bottom))
+  )
+  (gr_text "A5" (at 225.183 124.084 90) (layer "F.SilkS")
+    (effects (font (size 1.5 1.5) (thickness 0.3)))
+  )
+  (gr_text "S5" (at 249.059 105.288) (layer "F.SilkS")
+    (effects (font (size 1.5 1.5) (thickness 0.15)) (justify left bottom))
   )
   (gr_text "+" (at 80.149 125.1) (layer "F.SilkS")
@@
     (effects (font (size 2 2) (thickness 0.3)) (justify left bottom))
   )
+  (gr_text "S9" (at 249.059 116.972) (layer "F.SilkS")
+    (effects (font (size 1.5 1.5) (thickness 0.15)) (justify left bottom))
+  )
   (gr_text "SER" (at 174.129 71.76) (layer "F.SilkS")
     (effects (font (size 2 2) (thickness 0.3)) (justify bottom))
   )
+  (gr_text "A0" (at 225.183 92.588 90) (layer "F.SilkS")
+    (effects (font (size 1.5 1.5) (thickness 0.3)))
+  )
   (gr_text "R" (at 174.129 67.315) (layer "F.SilkS")
     (effects (font (size 1.5 1.5) (thickness 0.3)) (justify bottom))
@@
     (effects (font (size 2 2) (thickness 0.3)) (justify left bottom))
   )
+  (gr_text "S" (at 252.869 88.016) (layer "F.SilkS")
+    (effects (font (size 1.2 1.2) (thickness 0.15)) (justify left bottom))
+  )
+  (gr_text "PropPlug\nProgramming\nHeader\n(#32201)" (at 71.894 79.3225) (layer "F.SilkS")
+    (effects (font (size 1 1) (thickness 0.15)) (justify bottom))
+  )
+  (gr_text "S13" (at 247.535 129.164) (layer "F.SilkS")
+    (effects (font (size 1.5 1.5) (thickness 0.15)) (justify left bottom))
+  )
+  (gr_text "S7" (at 249.059 110.368) (layer "F.SilkS")
+    (effects (font (size 1.5 1.5) (thickness 0.15)) (justify left bottom))
+  )
   (gr_text "S" (at 127.139 67.315) (layer "F.SilkS")
     (effects (font (size 1.5 1.5) (thickness 0.3)) (justify bottom))
   )
+  (gr_text "S15" (at 247.535 134.244) (layer "F.SilkS")
+    (effects (font (size 1.5 1.5) (thickness 0.15)) (justify left bottom))
+  )
   (gr_text "LED OUT" (at 125.869 71.125) (layer "F.SilkS")
     (effects (font (size 1.5 1.5) (thickness 0.3) bold) (justify bottom))
   )
+  (gr_text "A4" (at 225.183 117.988 90) (layer "F.SilkS")
+    (effects (font (size 1.5 1.5) (thickness 0.3)))
+  )
   (dimension (type aligned) (layer "Dwgs.User")

Commit message: Add Logo, cleanup
Parts:
- added G***: LOGO, MoreSymbols:Kevinbot3, F.Cu at (164.2, 126.1)
Other:
- board text added: "3"
- board text added: "5"
- board text added: "A"
- board text added: "I2C"
- board text added: "L"
- board text added: "ONE-WIRE"
