File: i2c.kicad_sch (KiCad schematic)
At the start: 4 parts, among them J35 Conn_01x05, J36 Conn_01x05, J37 Conn_01x05, J38 Conn_01x05

Commit message: Fix global labels
Parts:
- renumbered J35 to J22, J37 to J23, J36 to J24, J38 to J25
Changed lines of the file:
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@@
 		(dnp no)
 		(fields_autoplaced yes)
-		(property "Reference" "J36"
+		(property "Reference" "J24"
 			(at 161.29 100.965 0)
 			(effects
@@
 			(project "P2 Kevinbot Board"
 				(path "/362ca48c-0b77-4943-b8b3-fc15ab97f30d/d951f0df-5c9d-49c8-96c9-1d29a8915b41"
-					(reference "J36")
+					(reference "J24")
 					(unit 1)
 				)
@@
 		(dnp no)
 		(fields_autoplaced yes)
-		(property "Reference" "J37"
+		(property "Reference" "J23"
 			(at 139.7 116.205 0)
 			(effects
@@
 			(project "P2 Kevinbot Board"
 				(path "/362ca48c-0b77-4943-b8b3-fc15ab97f30d/d951f0df-5c9d-49c8-96c9-1d29a8915b41"
-					(reference "J37")
+					(reference "J23")
 					(unit 1)
 				)
@@
 		(dnp no)
 		(fields_autoplaced yes)
-		(property "Reference" "J38"
+		(property "Reference" "J25"
 			(at 161.29 114.935 0)
 			(effects
@@
 			(project "P2 Kevinbot Board"
 				(path "/362ca48c-0b77-4943-b8b3-fc15ab97f30d/d951f0df-5c9d-49c8-96c9-1d29a8915b41"
-					(reference "J38")
+					(reference "J25")
 					(unit 1)
 				)
@@
 		(dnp no)
 		(fields_autoplaced yes)
-		(property "Reference" "J35"
+		(property "Reference" "J22"
 			(at 139.7 100.965 0)
 			(effects
@@
 			(project "P2 Kevinbot Board"
 				(path "/362ca48c-0b77-4943-b8b3-fc15ab97f30d/d951f0df-5c9d-49c8-96c9-1d29a8915b41"
-					(reference "J35")
-					(unit 1)
-				)
+					(reference "J22")
+					(unit 1)
+				)

Commit message: Add mfr part numbers and datasheets to all
Parts:
- J22, J23, J24, J25: Part Number (none) -> B5B-XH-A
Changed lines of the file:
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@@
 			)
 		)
-		(property "Datasheet" "~"
+		(property "Datasheet" "https://www.jst-mfg.com/product/pdf/eng/eXH.pdf"
 			(at 158.75 100.33 0)
 			(effects
@@
 		)
 		(property "Description" "Generic connector, single row, 01x05, script generated (kicad-library-utils/schlib/autogen/connector/)"
+			(at 158.75 100.33 0)
+			(effects
+				(font
+					(size 1.27 1.27)
+				)
+				(hide yes)
+			)
+		)
+		(property "Part Number" "B5B-XH-A"
 			(at 158.75 100.33 0)
 			(effects
@@
 			)
 		)
-		(property "Datasheet" "~"
-			(at 137.16 115.57 0)
-			(effects
-				(font
-					(size 1.27 1.27)
-				)
-				(hide yes)
-			)
-		)
-		(property "Description" "Generic connector, single row, 01x05, script generated (kicad-library-utils/schlib/autogen/connector/)"
+		(property "Datasheet" "https://www.jst-mfg.com/product/pdf/eng/eXH.pdf"
+			(at 137.16 115.57 0)
+			(effects
+				(font
+					(size 1.27 1.27)
+				)
+				(hide yes)
+			)
+		)
+		(property "Description" "Generic connector, single row, 01x05, script generated (kicad-library-utils/schlib/autogen/connector/)"
+			(at 137.16 115.57 0)
+			(effects
+				(font
+					(size 1.27 1.27)
+				)
+				(hide yes)
+			)
+		)
+		(property "Part Number" "B5B-XH-A"
 			(at 137.16 115.57 0)
 			(effects
@@
 			)
 		)
-		(property "Datasheet" "~"
-			(at 158.75 115.57 0)
-			(effects
-				(font
-					(size 1.27 1.27)
-				)
-				(hide yes)
-			)
-		)
-		(property "Description" "Generic connector, single row, 01x05, script generated (kicad-library-utils/schlib/autogen/connector/)"
+		(property "Datasheet" "https://www.jst-mfg.com/product/pdf/eng/eXH.pdf"
+			(at 158.75 115.57 0)
+			(effects
+				(font
+					(size 1.27 1.27)
+				)
+				(hide yes)
+			)
+		)
+		(property "Description" "Generic connector, single row, 01x05, script generated (kicad-library-utils/schlib/autogen/connector/)"
+			(at 158.75 115.57 0)
+			(effects
+				(font
+					(size 1.27 1.27)
+				)
+				(hide yes)
+			)
+		)
+		(property "Part Number" "B5B-XH-A"
 			(at 158.75 115.57 0)
 			(effects
@@
 			)
 		)
-		(property "Datasheet" "~"
-			(at 137.16 100.33 0)
-			(effects
-				(font
-					(size 1.27 1.27)
-				)
-				(hide yes)
-			)
-		)
-		(property "Description" "Generic connector, single row, 01x05, script generated (kicad-library-utils/schlib/autogen/connector/)"
-			(at 137.16 100.33 0)
-			(effects
+		(property "Datasheet" "https://www.jst-mfg.com/product/pdf/eng/eXH.pdf"
+			(at 137.16 100.33 0)
+			(effects
+				(font
+					(size 1.27 1.27)
+				)
+				(hide yes)
+			)
+		)
+		(property "Description" "Generic connector, single row, 01x05, script generated (kicad-library-utils/schlib/autogen/connector/)"
+			(at 137.16 100.33 0)
+			(effects
+				(font
+					(size 1.27 1.27)
+				)
+				(hide yes)
+			)
+		)
+		(property "Part Number" "B5B-XH-A"
+			(at 137.16 100.33 0)
+			(effects
