File: leds.kicad_sch (KiCad schematic)
At the start: 5 parts, among them J21 Conn_01x02, J32 Conn_01x02, Q2 IRLML6402, U4 TC4427

Commit message: Fix major mosfet wiring error
Connections:
- net GND: now also J32.1 (Pin_1); no longer Q2.2 (S)
- net LED_PWR: now also Q2.2 (S); no longer J32.2 (Pin_2)
- net at Q2.3 (D): now also J32.2 (Pin_2); no longer J32.1 (Pin_1)
Other:
- moved on the sheet: J32
Changed lines of the file:
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@@
+	(wire
+		(pts
+			(xy 236.22 104.14) (xy 222.25 104.14)
+		)
+		(stroke
+			(width 0)
+			(type default)
+		)
+	)
 	(wire
 		(pts
@@
 	(wire
 		(pts
-			(xy 222.25 83.82) (xy 238.76 83.82)
+			(xy 151.13 88.9) (xy 161.29 88.9)
 		)
 		(stroke
@@
 	(wire
 		(pts
-			(xy 151.13 88.9) (xy 161.29 88.9)
+			(xy 222.25 97.79) (xy 222.25 104.14)
 		)
 		(stroke
@@
 		)
 	)
-	(wire
-		(pts
-			(xy 222.25 83.82) (xy 222.25 87.63)
-		)
-		(stroke
-			(width 0)
-			(type default)
-		)
-	)
 	(global_label "BODY_LED"
 		(shape input)
@@
 	(global_label "LED_PWR"
 		(shape input)
-		(at 238.76 86.36 180)
+		(at 222.25 87.63 90)
 		(fields_autoplaced yes)
 		(effects
@@
 				(size 1.27 1.27)
 			)
-			(justify right)
+			(justify left)
 		)
 		(property "Intersheetrefs" "${INTERSHEET_REFS}"
-			(at 227.3687 86.36 0)
-			(effects
-				(font
-					(size 1.27 1.27)
-				)
-				(justify right)
+			(at 222.25 76.2387 90)
+			(effects
+				(font
+					(size 1.27 1.27)
+				)
+				(justify left)
 				(hide yes)
 			)
@@
 	)
 	(symbol
-		(lib_id "Transistor_FET:IRLML6402")
-		(at 219.71 92.71 0)
+		(lib_id "power:GND")
+		(at 236.22 101.6 270)
 		(unit 1)
 		(exclude_from_sim no)
@@
 		(dnp no)
 		(fields_autoplaced yes)
+		(property "Reference" "#PWR030"
+			(at 229.87 101.6 0)
+			(effects
+				(font
+					(size 1.27 1.27)
+				)
+				(hide yes)
+			)
+		)
+		(property "Value" "GND"
+			(at 232.41 101.5999 90)
+			(effects
+				(font
+					(size 1.27 1.27)
+				)
+				(justify right)
+			)
+		)
+		(property "Footprint" ""
+			(at 236.22 101.6 0)
+			(effects
+				(font
+					(size 1.27 1.27)
+				)
+				(hide yes)
+			)
+		)
+		(property "Datasheet" ""
+			(at 236.22 101.6 0)
+			(effects
+				(font
+					(size 1.27 1.27)
+				)
+				(hide yes)
+			)
+		)
+		(property "Description" "Power symbol creates a global label with name \"GND\" , ground"
+			(at 236.22 101.6 0)
+			(effects
+				(font
+					(size 1.27 1.27)
+				)
+				(hide yes)
+			)
+		)
+		(pin "1"
+		)
+		(instances
+			(project "P2 Kevinbot Board"
+				(path "/362ca48c-0b77-4943-b8b3-fc15ab97f30d/971de258-84b3-438c-84b6-ee44796701a6"
+					(reference "#PWR030")
+					(unit 1)
+				)
+			)
+		)
+	)
+	(symbol
+		(lib_id "Transistor_FET:IRLML6402")
+		(at 219.71 92.71 0)
+		(mirror x)
+		(unit 1)
+		(exclude_from_sim no)
+		(in_bom yes)
+		(on_board yes)
+		(dnp no)
+		(fields_autoplaced yes)
 		(property "Reference" "Q2"
-			(at 226.06 91.4399 0)
+			(at 226.06 93.9801 0)
 			(effects
 				(font
@@
 		)
 		(property "Value" "IRLML6402"
-			(at 226.06 93.9799 0)
+			(at 226.06 91.4401 0)
 			(effects
 				(font
@@
 		)
 		(property "Footprint" "Package_TO_SOT_SMD:SOT-23"
-			(at 224.79 94.615 0)
+			(at 224.79 90.805 0)
 			(effects
 				(font
@@
 		)
 		(property "Datasheet" "https://www.infineon.com/dgdl/irlml6402pbf.pdf?fileId=5546d462533600a401535668d5c2263c"
-			(at 224.79 96.52 0)
+			(at 224.79 88.9 0)
 			(effects
 				(font
@@
 	(symbol
 		(lib_id "Connector_Generic:Conn_01x02")
-		(at 243.84 83.82 0)
+		(at 241.3 101.6 0)
 		(unit 1)
 		(exclude_from_sim yes)
@@
 		(fields_autoplaced yes)
 		(property "Reference" "J32"
-			(at 246.38 83.8199 0)
+			(at 243.84 101.5999 0)
 			(effects
 				(font
@@
 		)
 		(property "Value" "Conn_01x02"
-			(at 246.38 86.3599 0)
+			(at 243.84 104.1399 0)
 			(effects
 				(font
@@
 		)
 		(property "Footprint" "Connector_JST:JST_XH_B2B-XH-A_1x02_P2.50mm_Vertical"
-			(at 243.84 83.82 0)
+			(at 241.3 101.6 0)
 			(effects
 				(font
@@
 		)
 		(property "Datasheet" "https://www.jst-mfg.com/product/pdf/eng/eXH.pdf"
-			(at 243.84 83.82 0)
+			(at 241.3 101.6 0)
 			(effects
 				(font
@@
 		)
 		(property "Description" "Generic connector, single row, 01x02, script generated (kicad-library-utils/schlib/autogen/connector/)"
-			(at 243.84 83.82 0)
+			(at 241.3 101.6 0)
 			(effects
 				(font
@@
 		)
 		(property "Part Number" "B2B-XH-A"
-			(at 243.84 83.82 0)
+			(at 241.3 101.6 0)
 			(effects
 				(font
@@
 					(unit 1)
 				)
-			)
-		)
-	)
-	(symbol
-		(lib_id "power:GND")
-		(at 222.25 97.79 0)
-		(unit 1)
-		(exclude_from_sim no)
-		(in_bom yes)
-		(on_board yes)
-		(dnp no)
-		(property "Reference" "#PWR030"
-			(at 222.25 104.14 0)
-			(effects
-				(font
-					(size 1.27 1.27)
-				)
-				(hide yes)
-			)
-		)
-		(property "Value" "GND"
-			(at 222.25 102.87 0)
-			(effects
-				(font
-					(size 1.27 1.27)
-				)
-			)
-		)
-		(property "Footprint" ""
-			(at 222.25 97.79 0)
-			(effects
-				(font
-					(size 1.27 1.27)
-				)
-				(hide yes)
-			)
-		)
-		(property "Datasheet" ""
-			(at 222.25 97.79 0)
-			(effects
-				(font
-					(size 1.27 1.27)
-				)
-				(hide yes)
-			)
-		)
-		(property "Description" "Power symbol creates a global label with name \"GND\" , ground"
-			(at 222.25 97.79 0)
-			(effects
-				(font
-					(size 1.27 1.27)
-				)
-				(hide yes)
-			)
-		)
-		(pin "1"
-		)
-		(instances
-			(project "P2 Kevinbot Board"
-				(path "/362ca48c-0b77-4943-b8b3-fc15ab97f30d/971de258-84b3-438c-84b6-ee44796701a6"
-					(reference "#PWR030")
-					(unit 1)
-				)

Commit message: Use tc4427 for RSL OUT, first commit for RevB
Parts:
- removed Q2: IRLML6402, Package_TO_SOT_SMD:SOT-23, symbol Transistor_FET:IRLML6402
- removed R26: 680R, Resistor_SMD:R_0603_1608Metric, symbol Device:R
Connections:
- net IN_RSL: now also U4.4 (INB)
- net RSL_LED: now reaches J32.2 (Pin_2)
- net RSL_LED: now also U4.5 (OUTB)
- no-connect marks 2 -> 0
