File: buzzout.kicad_sch (KiCad schematic)
At the start: 2 parts

Commit message: Buzzer
Parts:
- added J4: Conn_01x02_Pin, Connector_Molex:Molex_Nano-Fit_105309-xx03_1x03_P2.50mm_Vertical, symbol Connector:Conn_01x03_Pin
- added Q2: IRLML6402, Package_TO_SOT_SMD:SOT-23, symbol Transistor_FET:IRLML6402
- added U5: TC4426xOA, Package_SO:SOIC-8_3.9x4.9mm_P1.27mm, symbol Driver_FET:TC4426xOA
Connections:
- net BZ_OUT: now reaches JP4.1 (A)
- net BZ_OUT: now also J4.2 (Pin_2), Q2.3 (D)
- net GND: now reaches BZ1.2 (-)
- net GND: now also J4.1 (Pin_1), U5.3 (GND)
- new net: Q2.1 (G), U5.7 (~{OUT_A})
- new net SIG: U5.2 (IN_A)
- new net VIN: J4.3 (Pin_3), Q2.2 (S), U5.6 (VDD)
- no-connect marks 0 -> 2
