File: buck.kicad_sch (KiCad schematic)
At the start: 26 parts, among them Q5 CSD18543Q3A, Q6 CSD18543Q3A

Commit message: pcb, buck: cleanup, add 7070 inductor DNP footprint
Parts:
- added L2: 6.8uH 11.5A, Inductor_Local:L_Coilcraft_XAL7070-XXX-NOSILK, symbol Device:L_Iron
- L1: Part Number (none) -> SRP1265A-6R8M
Connections:
- net 5VOUT: now also L2.2
- net at C19.1, L1.1, Q5.1 (S)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: now also L2.1
Changed lines of the file:
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@@
+	)
+	(junction
+		(at 190.5 83.82)
+		(diameter 0)
+		(color 0 0 0 0)
 	)
 	(junction
@@
 	)
 	(junction
+		(at 198.12 83.82)
+		(diameter 0)
+		(color 0 0 0 0)
+	)
+	(junction
 		(at 248.92 83.82)
 		(diameter 0)
@@
 	(wire
 		(pts
+			(xy 198.12 83.82) (xy 198.12 92.71)
+		)
+		(stroke
+			(width 0)
+			(type default)
+		)
+	)
+	(wire
+		(pts
 			(xy 168.91 83.82) (xy 168.91 91.44)
 		)
@@
 		(pts
 			(xy 83.82 73.66) (xy 83.82 71.12)
+		)
+		(stroke
+			(width 0)
+			(type default)
+		)
+	)
+	(wire
+		(pts
+			(xy 190.5 83.82) (xy 190.5 92.71)
 		)
 		(stroke
@@
 			)
 		)
-		(property "Part Number" ""
+		(property "Part Number" "SRP1265A-6R8M"
 			(at 194.31 83.82 90)
 			(effects
@@
 					(unit 1)
 				)
+			)
+		)
+	)
+	(symbol
+		(lib_id "Device:L_Iron")
+		(at 194.31 92.71 90)
+		(unit 1)
+		(exclude_from_sim no)
+		(in_bom yes)
+		(on_board yes)
+		(dnp yes)
+		(property "Reference" "L2"
+			(at 194.31 94.488 90)
+			(effects
+				(font
+					(size 1.27 1.27)
+				)
+			)
+		)
+		(property "Value" "6.8uH 11.5A"
+			(at 194.31 97.028 90)
+			(effects
+				(font
+					(size 1.27 1.27)
+				)
+			)
+		)
+		(property "Footprint" "Inductor_Local:L_Coilcraft_XAL7070-XXX-NOSILK"
+			(at 194.31 92.71 0)
+			(effects
+				(font
+					(size 1.27 1.27)
+				)
+				(hide yes)
+			)
+		)
+		(property "Datasheet" "~"
+			(at 194.31 92.71 0)
+			(effects
+				(font
+					(size 1.27 1.27)
+				)
+				(hide yes)
+			)
+		)
+		(property "Description" "Inductor with iron core"
+			(at 194.31 92.71 0)
+			(effects
+				(font
+					(size 1.27 1.27)
+				)
+				(hide yes)
+			)
+		)
+		(property "Part Number" "XAL7070-682MEC"
+			(at 194.31 92.71 90)
+			(effects
+				(font
+					(size 1.27 1.27)
+				)
+				(hide yes)
+			)
+		)
+		(pin "2"
+		)
+		(pin "1"
+		)
+		(instances
+			(project "P2 Kevinbot Board"
+				(path "/362ca48c-0b77-4943-b8b3-fc15ab97f30d/083e4746-c54f-4ebf-8db7-bc4666178b1b/51854cd4-d173-4e7e-b3ec-d45904214b7f"
+					(reference "L2")
+					(unit 1)
+				)

Commit message: sch: erc
Other:
- moved on the sheet: R49

Commit message: part number fix
Parts:
- C17: Part Number (none) -> C0603C563J4RACTU; Part Number1 C0603C563J4RACTU -> (none)
Changed lines of the file:
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@@
 			)
 		)
-		(property "Part Number1" "C0603C563J4RACTU"
+		(property "Part Number" "C0603C563J4RACTU"
 			(at 39.37 99.06 0)
 			(effects
